File: SmartiePiHub.sch (KiCad schematic (older format))
At the start: 97 parts, among them CN1 SX1238_TRX_HEADER, CN2 ZIGBEE_TRX_HEADER, CN3 ZWAVE_TRX_HEADER, CN4 USB_C_Plug_USB2.0, CN5 RPI, SW1 SW_Push, SW2 SW_Push, SW3 SW_SPST, U1 WM8960, U2 MCP73833T-AMMF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

Commit message: adding more footprints. created netlist
Parts:
- CN1: footprint (none) -> SmartiePiHub:sx1238_trx
- CN2, CN3: footprint (none) -> Connector_PinSocket_2.54mm:PinSocket_2x06_P2.54mm_Vertical
Changed lines of the file:
@@
 F 0 "CN1" H 1850 4500 50  0000 C CNN
 F 1 "SX1238_TRX_HEADER" H 1900 5626 50  0000 C CNN
-F 2 "" H 1850 5100 50  0001 C CNN
+F 2 "SmartiePiHub:sx1238_trx" H 1850 5100 50  0001 C CNN
 F 3 "~" H 1850 5100 50  0001 C CNN
 	1    1850 5100
@@
 F 0 "CN3" H 4100 6467 50  0000 C CNN
 F 1 "ZWAVE_TRX_HEADER" H 4100 6376 50  0000 C CNN
-F 2 "" H 4050 6050 50  0001 C CNN
+F 2 "Connector_PinSocket_2.54mm:PinSocket_2x06_P2.54mm_Vertical" H 4050 6050 50  0001 C CNN
 F 3 "~" H 4050 6050 50  0001 C CNN
 	1    4050 6050
@@
 F 0 "CN2" H 4100 5517 50  0000 C CNN
 F 1 "ZIGBEE_TRX_HEADER" H 4100 5426 50  0000 C CNN
-F 2 "" H 4050 5100 50  0001 C CNN
+F 2 "Connector_PinSocket_2.54mm:PinSocket_2x06_P2.54mm_Vertical" H 4050 5100 50  0001 C CNN
 F 3 "~" H 4050 5100 50  0001 C CNN
 	1    4050 5100
